Commit message: Latest UR5 models and code

File: UR5/urdf/ur5.urdf (robot description, URDF)
Before this commit: robot sisbot, 11 links, 10 joints
Links:
- removed link base_link
- removed link ee_link
- removed link forearm_link
- removed link left_gripper
- removed link right_gripper
- removed link shoulder_link
- removed link upper_arm_link
- removed link wrist_1_link
- removed link wrist_2_link
- removed link wrist_3_link
- added link ur5/base_link; visual mesh filename=../meshes/ur_description/meshes/ur5/visual/base.dae
- added link ur5/ee_link; collision box size=0.01 0.01 0.01
- added link ur5/forearm_link; visual mesh filename=../meshes/ur_description/meshes/ur5/visual/forearm.dae
- added link ur5/left_gripper, mass .2; collision box size=0.02 0.02 0.15; visual mesh filename=../meshes/ur5/visual/l_gripper_tip_scaled.stl scale=1 1 1
- added link ur5/right_gripper, mass .2; collision box size=0.02 0.02 0.15; visual mesh filename=../meshes/ur5/visual/l_gripper_tip_scaled.stl scale=1 1 1
- added link ur5/shoulder_link; visual mesh filename=../meshes/ur_description/meshes/ur5/visual/shoulder.dae
- added link ur5/upper_arm_link; visual mesh filename=../meshes/ur_description/meshes/ur5/visual/upperarm.dae
- added link ur5/wrist_1_link; visual mesh filename=../meshes/ur_description/meshes/ur5/visual/wrist1.dae
- added link ur5/wrist_2_link; visual mesh filename=../meshes/ur_description/meshes/ur5/visual/wrist2.dae
- added link ur5/wrist_3_link; visual mesh filename=../meshes/ur_description/meshes/ur5/visual/wrist3.dae
Joints:
- joint ee_fixed_joint: child ee_link -> ur5/ee_link; parent wrist_3_link -> ur5/wrist_3_link
- joint elbow_joint: child forearm_link -> ur5/forearm_link; limit lower=-3.14159265359 upper=3.14159265359 effort=300.0 velocity=10 -> lower=-3.14159265 upper=3.14159265 effort=150.0 velocity=3.15; parent upper_arm_link -> ur5/upper_arm_link
- joint left_gripper_motor: child left_gripper -> ur5/left_gripper; parent wrist_3_link -> ur5/wrist_3_link
- joint right_gripper_motor: child right_gripper -> ur5/right_gripper; parent wrist_3_link -> ur5/wrist_3_link
- joint shoulder_lift_joint: child upper_arm_link -> ur5/upper_arm_link; limit lower=-3.14159265359 upper=3.14159265359 effort=300.0 velocity=10 -> lower=-3.14159265 upper=3.14159265 effort=150.0 velocity=3.15; origin xyz=0.0 0.13585 0.0 rpy=0.0 4.8 0.0 -> xyz=0.0 0.13585 0.0 rpy=0.0 1.570796325 0.0; parent shoulder_link -> ur5/shoulder_link
- joint shoulder_pan_joint: child shoulder_link -> ur5/shoulder_link; limit lower=-3.14159265359 upper=3.14159265359 effort=300.0 velocity=10 -> lower=-3.14159265 upper=3.14159265 effort=150.0 velocity=3.15; origin xyz=0.0 0.0 0.089159 rpy=0.0 0.0 3.14 -> xyz=0.0 0.0 0.089159 rpy=0.0 0.0 0.0; parent base_link -> ur5/base_link
- joint world_joint: child base_link -> ur5/base_link; origin xyz=0.0 0.0 0.1 rpy=0.0 0.0 0 -> xyz=0.0 0.0 0 rpy=0.0 0.0 0
- joint wrist_1_joint: child wrist_1_link -> ur5/wrist_1_link; limit lower=-3.14159265359 upper=3.14159265359 effort=300.0 velocity=10 -> lower=-3.14159265 upper=3.14159265 effort=28.0 velocity=3.2; origin xyz=0.0 0.0 0.39225 rpy=0.0 1.57079632679 0.0 -> xyz=0.0 0.0 0.39225 rpy=0.0 1.570796325 0.0; parent forearm_link -> ur5/forearm_link
- joint wrist_2_joint: child wrist_2_link -> ur5/wrist_2_link; limit lower=-3.14159265359 upper=3.14159265359 effort=300.0 velocity=10 -> lower=-3.14159265 upper=3.14159265 effort=28.0 velocity=3.2; parent wrist_1_link -> ur5/wrist_1_link
- joint wrist_3_joint: child wrist_3_link -> ur5/wrist_3_link; limit lower=-3.14159265359 upper=3.14159265359 effort=300.0 velocity=10 -> lower=-3.14159265 upper=3.14159265 effort=28.0 velocity=3.2; parent wrist_2_link -> ur5/wrist_2_link
