Commit message: Added UR5 Pick-n-Place Simulation - Fixes Reqd

File: src/meshes/small_block.urdf (robot description, URDF)
Before this commit: robot block_2, 1 links, 0 joints
Links:
- link block_2_base_link: geometry collision box size=0.05 0.05 0.1; visual box size=0.05 0.05 0.1

Commit message: Added two UR5 robots and updated the simulation

File: src/meshes/small_block.urdf (robot description, URDF)
Before this commit: robot block_2, 1 links, 0 joints
Links:
- link block_2_base_link: geometry collision box size=0.05 1 0.1; visual box size=0.05 1 0.1
